Commit message: yeyeyeye

File: description/robot_core.xacro (robot description, xacro)
@@ -13,5 +13,5 @@
         <color rgba="0 0 0 1" />
     </material>
-    <link name="base link">
+    <link name="base_link">
     </link>
     <joint name="chassis_joint" type="fixed">

Commit message: added wheels i think

File: description/robot_core.xacro (robot description, xacro)
@@ -13,6 +13,8 @@
         <color rgba="0 0 0 1" />
     </material>
+    <!-- BASE LINK-->
     <link name="base_link">
     </link>
+    <!-- CHASSIS LINK -->
     <joint name="chassis_joint" type="fixed">
         <parent link="base_link"/>
@@ -29,3 +31,33 @@
         </visual>
     </link>
+<!-- LEFT WHEEL LINK -->
+<joint name="left_wheel_joint" type="continuous">
+    <parent link="base_link"/>
+    <child link="left_wheel"/>
+    <origin xyz="0 0.175 0" rpy="-${pi/2} 0 0"/>
+    <axis xyz="0 0 1"/>
+</joint>
+<link name="left_wheel">
+    <visual>
+        <geometry>
+            <cylinder radius="0.05" length="0.04"/>
+        </geometry>
+        <material name="blue"/>
+    </visual>
+</link>
+<!-- RIGHT WHEEL LINK -->
+<joint name="right_wheel_joint" type="continuous">
+    <parent link="base_link"/>
+    <child link="right_wheel"/>
+    <origin xyz="0 -0.175 0" rpy="${pi/2} 0 0"/>
+    <axis xyz="0 0 -1"/>
+</joint>
+<link name="right_wheel">
+    <visual>
+        <geometry>
+            <cylinder radius="0.05" length="0.04"/>
+        </geometry>
+        <material name="blue"/>
+    </visual>
+</link>
 </robot>

Commit message: caster wheel added?

File: description/robot_core.xacro (robot description, xacro)
@@ -61,3 +61,17 @@
     </visual>
 </link>
+<!-- CASTER WHEEL LINK-->
+<joint name="caster_wheel_link" type="fixed">
+    <parent link="chassis"/>
+    <child link="caster=wheel"/>
+    <origin xyz="0.24 0 0"/>
+</joint>
+    <link name="caster_wheel">
+        <visual>
+            <geometry>
+                <sphere radius="0.05"/>
+            </geometry>
+            <material name="black"/>
+        </visual>
+    </link>
 </robot>

Commit message: found typo

File: description/robot_core.xacro (robot description, xacro)
@@ -64,5 +64,5 @@
 <joint name="caster_wheel_link" type="fixed">
     <parent link="chassis"/>
-    <child link="caster=wheel"/>
+    <child link="caster_wheel"/>
     <origin xyz="0.24 0 0"/>
 </joint>

Commit message: added collisions

File: description/robot_core.xacro (robot description, xacro)
@@ -30,4 +30,10 @@
             <material name="white"/>
         </visual>
+        <collision
+            <origin xyz="0.15 0 0.075"/>
+            <geometry>
+                <box size ="0.3 0.3 0.15"/>
+            </geometry>
+        </collision>
     </link>
 <!-- LEFT WHEEL LINK -->
@@ -45,4 +51,9 @@
         <material name="blue"/>
     </visual>
+    <collisoin>
+        <geometry>
+            <cylinder radius="0.05" length="0.04"/>
+        </geometry>
+    </collision>
 </link>
 <!-- RIGHT WHEEL LINK -->
@@ -60,4 +71,9 @@
         <material name="blue"/>
     </visual>
+    <collision>
+        <geometry>
+            <cylinder radius="0.05" length="0.04"/>
+        </geometry>
+    </collision>
 </link>
 <!-- CASTER WHEEL LINK-->
@@ -74,4 +90,9 @@
             <material name="black"/>
         </visual>
+        <collision>
+            <geometry>
+                <sphere radius="0.05"/>
+            </geometry>
+        </collision>
     </link>
 </robot>

Commit message: foudn typo

File: description/robot_core.xacro (robot description, xacro)
@@ -30,5 +30,5 @@
             <material name="white"/>
         </visual>
-        <collision
+        <collision>
             <origin xyz="0.15 0 0.075"/>
             <geometry>

Commit message: found typo

File: description/robot_core.xacro (robot description, xacro)
@@ -51,5 +51,5 @@
         <material name="blue"/>
     </visual>
-    <collisoin>
+    <collision>
         <geometry>
             <cylinder radius="0.05" length="0.04"/>

Commit message: added inertia file and updated inertai code

File: description/robot_core.xacro (robot description, xacro)
@@ -1,4 +1,5 @@
 <?xml version="1.0"?>
 <robot xmlns:xacro="http://www.ros.org/wiki/xacro" >
+    <xacro:include filename="inertial_macros.xacro"/>
     <material name="white">
         <color rgba="1 1 1 1" />
@@ -36,4 +37,7 @@
             </geometry>
         </collision>
+        <xacro:intertial_box mass="0.5" x="0.3" y="0.3" z="0.15">
+            <origin xyz="0.15 0 0.075" rpy="0 0 0"/>
+        </xacro:intertial_box>
     </link>
 <!-- LEFT WHEEL LINK -->
@@ -56,4 +60,7 @@
         </geometry>
     </collision>
+    <xacro:inertial_cylinder mass="0.1" length="0.4" radius="0.05">
+        <origin xyz="0 0 0" rpy="0 0 0"/>
+    </xacro:inertial_cylinder>
 </link>
 <!-- RIGHT WHEEL LINK -->
@@ -76,4 +83,7 @@
         </geometry>
     </collision>
+    <xacro:inertial_cylinder mass="0.1" length="0.4" radius="0.05">
+        <origin xyz="0 0 0" rpy="0 0 0"/>
+    </xacro:inertial_cylinder>
 </link>
 <!-- CASTER WHEEL LINK-->
@@ -95,4 +105,7 @@
             </geometry>
         </collision>
+        <xacro:inertial_sphere mass="0.1" radius="0.05">
+            <origin xyz="0 0 0" rpy="0 0 0"/>
+            </xacro:inertial_sphere>
     </link>
 </robot>
